Commit message: 修改好摩擦力后可以正常前走

File: ros2_all_wheel_sim/urdf/all_wheel/ALL_WHEEL.urdf (robot description, URDF)
Before this commit: robot ALL_WHEEL, 9 links, 8 joints
Links:
- link front_link: geometry collision cylinder length=0.03 radius=0.035115; visual mesh filename=package://ros2_all_wheel_sim/meshes/all_wheel/front_link.STL
- link left_Link: geometry collision cylinder length=0.03 radius=0.035115; visual mesh filename=package://ros2_all_wheel_sim/meshes/all_wheel/left_Link.STL
- link right_Link: geometry collision cylinder length=0.03 radius=0.035115; visual mesh filename=package://ros2_all_wheel_sim/meshes/all_wheel/right_Link.STL
