Commit message: 优化先调整方向再运行，调整相机位置

File: src/ros2_all_wheel_sim/urdf/all_wheel/ALL_WHEEL.urdf (robot description, URDF)
Before this commit: robot ALL_WHEEL, 9 links, 8 joints
Joints:
- joint stereo_left_joint: origin xyz=-0.05 0.05 0.06 rpy=0 0 3.1415926 -> xyz=0.08 0.05 0.06 rpy=0 0 0
- joint stereo_right_joint: origin xyz=-0.05 -0.05 0.06 rpy=0 0 3.1415926 -> xyz=0.08 -0.05 0.06 rpy=0 0 0
